File: fsr_endstop.sch (EAGLE design)
At the start: 0 parts

Commit message: Schematic first rev complete
Parts:
- added +/-, -/+, FSR1, FSR1A, FSR2, FSR2A, FSR3, FSR3A, GND, IO1, IO2, IO3, SIG, VCC: PIN1.2MM, _sg_lib:PIN1.2MM
- added AVR1: AVR6, _sg_misc:AVR6
- added C1: 1uF, _sg_lib:CAP0603
- added D1, D2, D3, D4: (no value), _sg_lib:DIODE0603
- added LED1, LED2, LED3, LED4: LED0603, _sg_lib:LED0603
- added R1, R2, R3, R4: (no value), _sg_lib:RES0603
- added R5, R6, R7: 10k, _sg_lib:RES0603
- added U1: ATTINY461, _sg_misc:ATTINY461
Connections:
- new net GND: AVR1.6_GND, C1.P$1, D3.-, D4.-, FSR1A.P$1, FSR2A.P$1, FSR3A.P$1, GND.P$1, LED1.-, LED2.-, LED3.-, LED4.-, U1.16_AGND, U1.6_GND
- new net N$1: AVR1.4_MOSI, U1.1_PB0_MOSI/DI/SDA/OC1A#/PCINT8
- new net N$10: R4.P$1, U1.14_PA4_ADC3/ICP0/PCINT4
- new net N$11: R3.P$1, U1.13_PA5_ADC4/AIN2/PCINT5
- new net N$12: R2.P$1, U1.12_PA6_ADC5/AIN0/PCINT6
- new net N$13: R1.P$1, U1.11_PA7_ADC6/AIN1/PCINT7
- new net N$14: SIG.P$1, U1.4_PB3_OC1B/PCINT11
- new net N$15: IO1.P$1, U1.9_PB6_ADC9/INT0/T0/PCINT14
- new net N$16: IO2.P$1, U1.8_PB5_ADC6/OC1D/CLK0/XTAL2/PCINT13
- new net N$17: IO3.P$1, U1.7_PB4_ADC7/OC1D#/CLKI/XTAL1/PCINT12
- new net N$18: LED1.+, R1.P$2
- new net N$19: LED2.+, R2.P$2
- new net N$2: AVR1.1_MISO, U1.2_PB1_MISO/DO/OC1A/PCINT9
- new net N$20: LED3.+, R3.P$2
- new net N$21: LED4.+, R4.P$2
- new net N$3: -/+.P$1, D2.-, D3.+
- new net N$4: +/-.P$1, D1.-, D4.+
- new net N$5: AVR1.3_SCK, U1.3_PB2_SCK/USCK/SCL/OC1B#/PCINT10
- new net N$6: AVR1.5_RST, U1.10_PB7_ADC10/RESET#/PCINT15
- new net N$7: FSR1.P$1, R5.P$1, U1.20_PA0_ADC0/DI/SDA/PCINT0
- new net N$8: FSR2.P$1, R6.P$1, U1.19_PA1_ADC1/DO/PCINT1
- new net N$9: FSR3.P$1, R7.P$1, U1.18_PA2_ADC2/INT1/USCK/SCL/PCINT2
- new net V+: AVR1.2_VCC, C1.P$2, D1.+, D2.+, R5.P$2, R6.P$2, R7.P$2, U1.15_AVCC, U1.5_VCC, VCC.P$1
